Commit message: Add GPS plugin and antenna

File: urdf/turtlebot2.urdf (robot description, URDF)
Before this commit: robot turtlebot, 36 links, 35 joints
Links:
- added link gps_base_link, mass 0.001; collision cylinder length=0.15 radius=0.005; visual cylinder length=0.15 radius=0.005
Joints:
- added joint gps_joint: type fixed, parent base_link, child gps_base_link, origin xyz=-0.05 0 0.475 rpy=0 0 0, axis 0 1 0
